File: LightPanels/SBX_connector_outline.brd (EAGLE design)
At the start: 133 x 232.4 mm, 0 parts

Commit message: SBX_connector_outline board complete
Parts:
- added +12V, CI, CO, DI, DO, GND: WIREPADSMD2,54-5,08, wirepad:SMD2,54-5,08
- added C1, C10, C11, C12, C13, C14, C15, C16, C17, C18, C19, C2, C20, C21, C22, C23, C24, C25, C26, C27, C28, C29, C3, C30, C31, C32, C33, C34, C35, C36, C37, C38, C39, C4, C40, C41, C42, C43, C44, C45, C46, C47, C5, C6, C7, C8, C9: (no value), SparkFun-Capacitors:0603-CAP
- added C48, C49: 10uF, SparkFun-Retired:EIA3216
- added IC1: LM1084-ADJ, lm1084-adj-to263:TO263-3
- added U$1, U$10, U$11, U$12, U$13, U$14, U$15, U$16, U$17, U$18, U$19, U$2, U$20, U$21, U$22, U$23, U$24, U$25, U$26, U$27, U$28, U$29, U$3, U$30, U$31, U$32, U$33, U$34, U$35, U$36, U$37, U$38, U$39, U$4, U$40, U$41, U$42, U$43, U$44, U$45, U$46, U$47, U$5, U$6, U$7, U$8, U$9: APA1025050, jos-ph:APA102_5050
Connections:
- new net +12V: +12V.1, C49.A, IC1.3
- new net +5V: C1.1, C10.1, C11.1, C12.1, C13.1, C14.1, C15.1, C16.1, C17.1, C18.1, C19.1, C2.1, C20.1, C21.1, C22.1, C23.1, C24.1, C25.1, C26.1, C27.1, C28.1, C29.1, C3.1, C30.1, C31.1, C32.1, C33.1, C34.1, C35.1, C36.1, C37.1, C38.1, C39.1, C4.1, C40.1, C41.1, C42.1, C43.1, C44.1, C45.1, C46.1, C47.1, C48.A, C5.1, C6.1, C7.1, C8.1, C9.1, IC1.2, U$1.1, U$10.1, U$11.1, U$12.1, U$13.1, U$14.1, U$15.1, U$16.1, U$17.1, U$18.1, U$19.1, U$2.1, U$20.1, U$21.1, U$22.1, U$23.1, U$24.1, U$25.1, U$26.1, U$27.1, U$28.1, U$29.1, U$3.1, U$30.1, U$31.1, U$32.1, U$33.1, U$34.1, U$35.1, U$36.1, U$37.1, U$38.1, U$39.1, U$4.1, U$40.1, U$41.1, U$42.1, U$43.1, U$44.1, U$45.1, U$46.1, U$47.1, U$5.1, U$6.1, U$7.1, U$8.1, U$9.1
- new net GND: C1.2, C10.2, C11.2, C12.2, C13.2, C14.2, C15.2, C16.2, C17.2, C18.2, C19.2, C2.2, C20.2, C21.2, C22.2, C23.2, C24.2, C25.2, C26.2, C27.2, C28.2, C29.2, C3.2, C30.2, C31.2, C32.2, C33.2, C34.2, C35.2, C36.2, C37.2, C38.2, C39.2, C4.2, C40.2, C41.2, C42.2, C43.2, C44.2, C45.2, C46.2, C47.2, C48.C, C49.C, C5.2, C6.2, C7.2, C8.2, C9.2, GND.1, U$1.6, U$10.6, U$11.6, U$12.6, U$13.6, U$14.6, U$15.6, U$16.6, U$17.6, U$18.6, U$19.6, U$2.6, U$20.6, U$21.6, U$22.6, U$23.6, U$24.6, U$25.6, U$26.6, U$27.6, U$28.6, U$29.6, U$3.6, U$30.6, U$31.6, U$32.6, U$33.6, U$34.6, U$35.6, U$36.6, U$37.6, U$38.6, U$39.6, U$4.6, U$40.6, U$41.6, U$42.6, U$43.6, U$44.6, U$45.6, U$46.6, U$47.6, U$5.6, U$6.6, U$7.6, U$8.6, U$9.6
- new net N$1: U$1.3, U$2.4
- new net N$10: U$5.2, U$6.5
- new net N$11: U$6.3, U$7.4
- new net N$12: U$6.2, U$7.5
- new net N$13: U$7.3, U$8.4
- new net N$14: U$7.2, U$8.5
- new net N$15: U$8.3, U$9.4
- new net N$16: U$8.2, U$9.5
- new net N$17: U$10.4, U$9.3
- new net N$18: U$10.5, U$9.2
- new net N$19: U$10.3, U$11.4
- new net N$2: U$1.2, U$2.5
- new net N$20: U$10.2, U$11.5
- new net N$21: U$11.3, U$12.4
- new net N$22: U$11.2, U$12.5
- new net N$23: U$12.3, U$13.4
- new net N$24: U$12.2, U$13.5
- new net N$25: U$13.3, U$14.4
- new net N$26: U$13.2, U$14.5
- new net N$27: U$14.3, U$15.4
- new net N$28: U$14.2, U$15.5
- new net N$29: U$15.3, U$16.4
- new net N$3: U$2.3, U$3.4
- new net N$30: U$15.2, U$16.5
- new net N$31: U$16.3, U$17.4
- new net N$32: U$32.3, U$33.4
- new net N$33: U$17.3, U$18.4
- new net N$34: U$17.2, U$18.5
- new net N$35: U$18.3, U$19.4
- new net N$36: U$18.2, U$19.5
- new net N$37: U$19.3, U$20.4
- new net N$38: U$19.2, U$20.5
- new net N$39: U$20.3, U$21.4
- new net N$4: U$2.2, U$3.5
- new net N$40: U$20.2, U$21.5
- new net N$41: U$21.3, U$22.4
- new net N$42: U$21.2, U$22.5
- new net N$43: U$22.3, U$23.4
- new net N$44: U$22.2, U$23.5
- new net N$45: U$23.3, U$24.4
- new net N$46: U$23.2, U$24.5
- new net N$47: U$24.3, U$25.4
- new net N$48: U$24.2, U$25.5
- new net N$49: U$25.3, U$26.4
- new net N$5: U$3.3, U$4.4
- new net N$50: U$25.2, U$26.5
- new net N$51: U$26.3, U$27.4
- new net N$52: U$26.2, U$27.5
- new net N$53: U$27.3, U$28.4
- new net N$54: U$27.2, U$28.5
- new net N$55: U$28.3, U$29.4
- new net N$56: U$28.2, U$29.5
- new net N$57: U$29.3, U$30.4
- new net N$58: U$29.2, U$30.5
- new net N$59: U$30.3, U$31.4
- new net N$6: U$3.2, U$4.5
- new net N$60: U$30.2, U$31.5
- new net N$61: U$31.3, U$32.4
- new net N$62: U$31.2, U$32.5
- new net N$63: U$1.4, U$47.3
- new net N$64: U$1.5, U$47.2
- new net N$65: U$33.3, U$34.4
- new net N$66: U$16.2, U$17.5
- new net N$67: U$33.2, U$34.5
- new net N$68: U$34.3, U$35.4
- new net N$69: U$34.2, U$35.5
- new net N$7: U$4.3, U$5.4
- new net N$70: U$35.3, U$36.4
- new net N$71: U$35.2, U$36.5
- new net N$72: U$36.3, U$37.4
- new net N$73: U$36.2, U$37.5
- new net N$74: U$37.3, U$38.4
- new net N$75: U$37.2, U$38.5
- new net N$76: U$38.3, U$39.4
- new net N$77: U$38.2, U$39.5
- new net N$78: DO.1, U$39.3
- new net N$79: CO.1, U$39.2
- new net N$8: U$4.2, U$5.5
- new net N$80: U$40.3, U$41.4
- new net N$81: U$40.2, U$41.5
- new net N$82: U$41.3, U$42.4
- new net N$83: U$41.2, U$42.5
- new net N$84: U$42.3, U$43.4
- new net N$85: U$42.2, U$43.5
- new net N$86: U$43.3, U$44.4
- new net N$87: U$43.2, U$44.5
- new net N$88: U$44.3, U$45.4
- new net N$89: U$44.2, U$45.5
- new net N$9: U$5.3, U$6.4
- new net N$90: U$45.3, U$46.4
- new net N$91: U$45.2, U$46.5
- new net N$92: U$46.3, U$47.4
- new net N$93: U$46.2, U$47.5
- new net N$94: CI.1, U$40.5
- new net N$95: DI.1, U$40.4
- new net N$98: U$32.2, U$33.5
Routing:
- net GND: track 0.00 -> 203.1 mm, vias 0 -> 47
- net N$30: track 0.00 -> 59.5 mm
- net N$29: track 0.00 -> 59.0 mm
- net N$94: track 0.00 -> 27.4 mm, vias 0 -> 1
- net N$95: track 0.00 -> 26.2 mm, vias 0 -> 1
- net N$78: track 0.00 -> 21.0 mm, vias 0 -> 1
- net N$79: track 0.00 -> 18.4 mm, vias 0 -> 1
- net N$64: track 0.00 -> 17.6 mm
- net N$8: track 0.00 -> 16.3 mm
- net N$7: track 0.00 -> 16.3 mm
- net N$6: track 0.00 -> 16.2 mm
- net N$5: track 0.00 -> 16.2 mm
- net N$48: track 0.00 -> 15.6 mm
- net N$63: track 0.00 -> 14.0 mm
- net N$83: track 0.00 -> 13.5 mm
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- added copper zone on layer 1, net +5V
- added copper zone on layer 16, net GND
Other:
- outline, holes or cut-outs redrawn

Commit message: Clean up light panels. Remvoe names/values
Parts:
- moved C49 3.31 mm to (10.0, 122.6), turned to 180 degrees
- moved C48 0.35 mm to (15.4, 122.6)
- moved U$10 0.16 mm to (117.8, 58.9)
- moved U$19 0.16 mm to (131.3, 143.4)
- moved U$20 0.16 mm to (131.3, 160.3)
- moved U$21 0.16 mm to (131.3, 177.3)
- moved U$22 0.16 mm to (131.3, 194.3)
Routing:
- net GND: track 203.1 -> 203.7 mm
- net +12V: track 9.79 -> 9.25 mm
Other:
- board text added: "SBX Connector"
