File: LightPanels/SBX_connector_outline.sch (EAGLE design)
At the start: 0 parts

Commit message: SBX_connector_outline board complete
Parts:
- added +12V, CI, CO, DI, DO, GND: WIREPADSMD2,54-5,08, wirepad:WIREPADSMD2,54-5,08
- added C1, C10, C11, C12, C13, C14, C15, C16, C17, C18, C19, C2, C20, C21, C22, C23, C24, C25, C26, C27, C28, C29, C3, C30, C31, C32, C33, C34, C35, C36, C37, C38, C39, C4, C40, C41, C42, C43, C44, C45, C46, C47, C5, C6, C7, C8, C9: (no value), SparkFun-Capacitors:CAP0603-CAP
- added C48, C49: 10uF, SparkFun-Retired:10UF-TANT
- added IC1: LM1084-ADJ, lm1084-adj-to263:LM1084-ADJ
- added U$1, U$10, U$11, U$12, U$13, U$14, U$15, U$16, U$17, U$18, U$19, U$2, U$20, U$21, U$22, U$23, U$24, U$25, U$26, U$27, U$28, U$29, U$3, U$30, U$31, U$32, U$33, U$34, U$35, U$36, U$37, U$38, U$39, U$4, U$40, U$41, U$42, U$43, U$44, U$45, U$46, U$47, U$5, U$6, U$7, U$8, U$9: APA1025050, jos-ph:APA1025050
Connections:
- new net +12V: +12V.P, C49.+, IC1.IN
- new net +5V: C1.1, C10.1, C11.1, C12.1, C13.1, C14.1, C15.1, C16.1, C17.1, C18.1, C19.1, C2.1, C20.1, C21.1, C22.1, C23.1, C24.1, C25.1, C26.1, C27.1, C28.1, C29.1, C3.1, C30.1, C31.1, C32.1, C33.1, C34.1, C35.1, C36.1, C37.1, C38.1, C39.1, C4.1, C40.1, C41.1, C42.1, C43.1, C44.1, C45.1, C46.1, C47.1, C48.+, C5.1, C6.1, C7.1, C8.1, C9.1, IC1.OUT, U$1.VCC, U$10.VCC, U$11.VCC, U$12.VCC, U$13.VCC, U$14.VCC, U$15.VCC, U$16.VCC, U$17.VCC, U$18.VCC, U$19.VCC, U$2.VCC, U$20.VCC, U$21.VCC, U$22.VCC, U$23.VCC, U$24.VCC, U$25.VCC, U$26.VCC, U$27.VCC, U$28.VCC, U$29.VCC, U$3.VCC, U$30.VCC, U$31.VCC, U$32.VCC, U$33.VCC, U$34.VCC, U$35.VCC, U$36.VCC, U$37.VCC, U$38.VCC, U$39.VCC, U$4.VCC, U$40.VCC, U$41.VCC, U$42.VCC, U$43.VCC, U$44.VCC, U$45.VCC, U$46.VCC, U$47.VCC, U$5.VCC, U$6.VCC, U$7.VCC, U$8.VCC, U$9.VCC
- new net GND: C1.2, C10.2, C11.2, C12.2, C13.2, C14.2, C15.2, C16.2, C17.2, C18.2, C19.2, C2.2, C20.2, C21.2, C22.2, C23.2, C24.2, C25.2, C26.2, C27.2, C28.2, C29.2, C3.2, C30.2, C31.2, C32.2, C33.2, C34.2, C35.2, C36.2, C37.2, C38.2, C39.2, C4.2, C40.2, C41.2, C42.2, C43.2, C44.2, C45.2, C46.2, C47.2, C48.-, C49.-, C5.2, C6.2, C7.2, C8.2, C9.2, GND.P, U$1.GND, U$10.GND, U$11.GND, U$12.GND, U$13.GND, U$14.GND, U$15.GND, U$16.GND, U$17.GND, U$18.GND, U$19.GND, U$2.GND, U$20.GND, U$21.GND, U$22.GND, U$23.GND, U$24.GND, U$25.GND, U$26.GND, U$27.GND, U$28.GND, U$29.GND, U$3.GND, U$30.GND, U$31.GND, U$32.GND, U$33.GND, U$34.GND, U$35.GND, U$36.GND, U$37.GND, U$38.GND, U$39.GND, U$4.GND, U$40.GND, U$41.GND, U$42.GND, U$43.GND, U$44.GND, U$45.GND, U$46.GND, U$47.GND, U$5.GND, U$6.GND, U$7.GND, U$8.GND, U$9.GND
- new net N$1: U$1.DO, U$2.DI
- new net N$10: U$5.CO, U$6.CI
- new net N$11: U$6.DO, U$7.DI
- new net N$12: U$6.CO, U$7.CI
- new net N$13: U$7.DO, U$8.DI
- new net N$14: U$7.CO, U$8.CI
- new net N$15: U$8.DO, U$9.DI
- new net N$16: U$8.CO, U$9.CI
- new net N$17: U$10.DI, U$9.DO
- new net N$18: U$10.CI, U$9.CO
- new net N$19: U$10.DO, U$11.DI
- new net N$2: U$1.CO, U$2.CI
- new net N$20: U$10.CO, U$11.CI
- new net N$21: U$11.DO, U$12.DI
- new net N$22: U$11.CO, U$12.CI
- new net N$23: U$12.DO, U$13.DI
- new net N$24: U$12.CO, U$13.CI
- new net N$25: U$13.DO, U$14.DI
- new net N$26: U$13.CO, U$14.CI
- new net N$27: U$14.DO, U$15.DI
- new net N$28: U$14.CO, U$15.CI
- new net N$29: U$15.DO, U$16.DI
- new net N$3: U$2.DO, U$3.DI
- new net N$30: U$15.CO, U$16.CI
- new net N$31: U$16.DO, U$17.DI
- new net N$32: U$32.DO, U$33.DI
- new net N$33: U$17.DO, U$18.DI
- new net N$34: U$17.CO, U$18.CI
- new net N$35: U$18.DO, U$19.DI
- new net N$36: U$18.CO, U$19.CI
- new net N$37: U$19.DO, U$20.DI
- new net N$38: U$19.CO, U$20.CI
- new net N$39: U$20.DO, U$21.DI
- new net N$4: U$2.CO, U$3.CI
- new net N$40: U$20.CO, U$21.CI
- new net N$41: U$21.DO, U$22.DI
- new net N$42: U$21.CO, U$22.CI
- new net N$43: U$22.DO, U$23.DI
- new net N$44: U$22.CO, U$23.CI
- new net N$45: U$23.DO, U$24.DI
- new net N$46: U$23.CO, U$24.CI
- new net N$47: U$24.DO, U$25.DI
- new net N$48: U$24.CO, U$25.CI
- new net N$49: U$25.DO, U$26.DI
- new net N$5: U$3.DO, U$4.DI
- new net N$50: U$25.CO, U$26.CI
- new net N$51: U$26.DO, U$27.DI
- new net N$52: U$26.CO, U$27.CI
- new net N$53: U$27.DO, U$28.DI
- new net N$54: U$27.CO, U$28.CI
- new net N$55: U$28.DO, U$29.DI
- new net N$56: U$28.CO, U$29.CI
- new net N$57: U$29.DO, U$30.DI
- new net N$58: U$29.CO, U$30.CI
- new net N$59: U$30.DO, U$31.DI
- new net N$6: U$3.CO, U$4.CI
- new net N$60: U$30.CO, U$31.CI
- new net N$61: U$31.DO, U$32.DI
- new net N$62: U$31.CO, U$32.CI
- new net N$63: U$1.DI, U$47.DO
- new net N$64: U$1.CI, U$47.CO
- new net N$65: U$33.DO, U$34.DI
- new net N$66: U$16.CO, U$17.CI
- new net N$67: U$33.CO, U$34.CI
- new net N$68: U$34.DO, U$35.DI
- new net N$69: U$34.CO, U$35.CI
- new net N$7: U$4.DO, U$5.DI
- new net N$70: U$35.DO, U$36.DI
- new net N$71: U$35.CO, U$36.CI
- new net N$72: U$36.DO, U$37.DI
- new net N$73: U$36.CO, U$37.CI
- new net N$74: U$37.DO, U$38.DI
- new net N$75: U$37.CO, U$38.CI
- new net N$76: U$38.DO, U$39.DI
- new net N$77: U$38.CO, U$39.CI
- new net N$78: DO.P, U$39.DO
- new net N$79: CO.P, U$39.CO
- new net N$8: U$4.CO, U$5.CI
- new net N$80: U$40.DO, U$41.DI
- new net N$81: U$40.CO, U$41.CI
- new net N$82: U$41.DO, U$42.DI
- new net N$83: U$41.CO, U$42.CI
- new net N$84: U$42.DO, U$43.DI
- new net N$85: U$42.CO, U$43.CI
- new net N$86: U$43.DO, U$44.DI
- new net N$87: U$43.CO, U$44.CI
- new net N$88: U$44.DO, U$45.DI
- new net N$89: U$44.CO, U$45.CI
- new net N$9: U$5.DO, U$6.DI
- new net N$90: U$45.DO, U$46.DI
- new net N$91: U$45.CO, U$46.CI
- new net N$92: U$46.DO, U$47.DI
- new net N$93: U$46.CO, U$47.CI
- new net N$94: CI.P, U$40.CI
- new net N$95: DI.P, U$40.DI
- new net N$98: U$32.CO, U$33.CI
