File: CANShield/CANShield.brd (EAGLE design)
At the start: 114.3 x 133.3 mm, 115 parts, among them IC1 7805DT, IC2 74LVC2G125DCT, IC3 ILD213T, J2 POWERPOLE_POWER25A_HORIZONTAL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, Q1 MOSFET-NCHANNELFDD8780, Q11 IRLML6344TRPBF, Q13 IRLML6344TRPBF, Q14 IRLML6344TRPBF, Q2 MOSFET-NCHANNELFDD8780, Q3 MOSFET-NCHANNELFDD8780, Q4 MOSFET-NCHANNELFDD8780, Q5 MOSFET-NCHANNELFDD8780, Q6 MOSFET-NCHANNELFDD8780, Q7 MOSFET-NCHANNELBSS123LT1G, Q8 BSS123, Q9 IRLML6344TRPBF, U5 MCP2551, X2 SMKDSP_1,5/2, X3 SMKDSP_1,5/2, X4 SMKDSP_1,5/2, X5 SMKDSP_1,5/2

Commit message: Mostly done
Parts:
- C1, C4: value (none) -> 10uF
- C5: value (none) -> 0.1uF
- R22: value (none) -> 470R
- R31: value (none) -> 100R
- R32: value (none) -> 10K
- moved PRECHARGE_FUSE 10.2 mm to (0.00, 58.4)
- moved X4 8.89 mm to (-6.35, 47.0)
- moved IC3 7.62 mm to (26.7, 63.5)
- moved R23 6.35 mm to (31.8, 66.0)
- moved R26 6.35 mm to (21.6, 66.0)
- moved X2 6.35 mm to (-6.35, 33.0)
- moved R36 5.08 mm to (8.89, 47.0)
- moved R3 5.08 mm to (77.1, 61.0)
- moved R6 5.08 mm to (77.1, 66.0)
- moved R37 4.70 mm to (15.2, 53.0)
- moved R39 4.02 mm to (17.8, 52.1), turned to 90 degrees
- moved 74HC125M 3.81 mm to (27.4, 45.8)
- moved LM393M 3.81 mm to (17.3, 45.8)
- moved Q9 3.81 mm to (17.8, 27.9)
- moved R24 3.81 mm to (24.9, 53.5)
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Connections:
- net PRECHARGE_RESISTOR_IN renamed PRECHARGE_RESISTOR_IN_1
- net PRECHARGE_RESISTOR_IN1 renamed PRECHARGE_RESISTOR_IN_2
Routing:
- net 96V_IN_FUSED: track 41.9 -> 51.1 mm
- net CHARGE_2: track 37.9 -> 30.8 mm
- net N$5: track 9.77 -> 15.0 mm
- net N$3: track 9.74 -> 14.9 mm
- net N$2: track 22.3 -> 17.2 mm
- net N$17: track 22.1 -> 17.1 mm
- net CAP_CHARGE_REF: track 40.8 -> 35.9 mm
- net AGND: track 47.5 -> 51.8 mm, vias 6 -> 10
- net SBO_SENSE_2: track 52.5 -> 56.3 mm
- net N$34: track 2.81 -> 6.62 mm
- net N$32: track 3.23 -> 7.04 mm
- net +5V: track 274.6 -> 277.1 mm
- net CAP_CHARGE_V_CURR_1: track 11.2 -> 8.84 mm
- net CHARGE_1: track 36.1 -> 33.9 mm
- net SBO_SENSE_1: track 37.2 -> 38.5 mm
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Other:
- board text added: "+"
- board text added: "12V"
- board text added: "12V SUPPLY"
- board text added: "96V PACK"
- board text added: "B"
- board text added: "CAN"
- board text added: "CO"
- board text added: "CONTACTOR 1"
- board text added: "CONTACTOR 2"
- board text added: "DO"
- board text added: "FANS"
- board text added: "FANS PWM"
- board text added: "FANS RGB"
- board text added: "G"
- board text added: "GND"
- board text added: "H"
- board text added: "IN"
- board text added: "L"
- board text added: "ON"
- board text added: "ON SWITCH"
- board text added: "PACK RGB"
- board text added: "PRECHARGE OUT"
- board text added: "PRECHARGE R"
- board text added: "PWM"
- board text added: "R"
- board text added: "R+"
- board text added: "R-"
- board text added: "SBO LOOP 1"
- board text added: "SBO LOOP 2"
- board text added: "SL"
- board text removed: "B+"
- board text removed: "B-"
- board text removed: "Reset"

Commit message: Feature complete pcb
Parts:
- added C10, C9: 0.1uF, SparkFun-Capacitors:0603-CAP
- added CAN1: SMKDSP_1,5/3, con-phoenix-smkdsp:SMKDSP_1,5/3
- added D12, D13: BAS40-04, diode:SOT23
- added F2: PTCTHERMISTOR1206, SparkFun-PowerIC:PTC-1206
- added IC6, IC7: 74LVC1G04DBV, 74xx-little-de:SOT23-5
- added R48, R49: 100R, SparkFun-Passives:0603-RES
- added X1: SMKDSP_1,5/2, con-phoenix-smkdsp:SMKDSP_1,5/2
- added X6: SMKDSP_1,5/4, con-phoenix-smkdsp:SMKDSP_1,5/4
- moved U$5 40.5 mm to (17.8, 72.4), turned to 270 degrees
- moved R26 13.0 mm to (34.3, 63.5), turned to 90 degrees
- moved PF2 12.8 mm to (67.3, -2.54)
- moved Q9 12.7 mm to (30.5, 27.9)
- moved R34 12.7 mm to (34.3, 27.9)
- moved CAN 11.4 mm to (-6.35, 96.5)
- moved PF1 8.63 mm to (86.4, -5.59), turned to 270 degrees
- moved CONTACTOR_1 7.62 mm to (29.2, -8.89)
- moved D7 7.41 mm to (2.54, 3.81), turned to 90 degrees
- moved IC3 7.18 mm to (31.8, 58.4), turned to 270 degrees
- moved R13 6.40 mm to (16.5, 76.3), turned to 180 degrees
- moved CONTACTOR_2 6.35 mm to (67.3, -8.89)
- moved D8 6.35 mm to (36.8, 21.6), turned to 270 degrees
- moved C3 5.08 mm to (9.53, 75.6)
- moved R12 5.08 mm to (11.4, 75.6)
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Connections:
- new net CONTACTOR_GND: U$7.10, U$8.10, X1.1
- new net N$36: R48.1, X6.4
- new net N$37: R49.1, X6.3
- new net N$47: F2.1, X6.2
- net +5V: now also C10.2, C9.2, D12.2, D13.2, D6.C, D7.C, F2.2, IC6.5, IC7.5, PRECHARGE_RELAY.1, PRECHARGE_RELAY1.1
- net 5V: no longer D6.C, D7.C, PRECHARGE_RELAY.1, PRECHARGE_RELAY1.1
- net AGND: no longer Q11.2, Q9.2, R34.2, R41.2
- net CHARGE_1: now also IC6.2, U$1.14/A0; no longer U$1.15/A1
- net CHARGE_2: now also IC7.2, U$1.15/A1; no longer U$1.14/A0
- net CONTACTOR_CLOSED_SENSE_1: now also U$1.18/A4; no longer U$1.16/A2
- net CONTACTOR_CLOSED_SENSE_2: now also U$1.19/A5; no longer U$1.17/A3
- net CONTACT_EN_1: now also IC6.4
- net CONTACT_EN_2: now also IC7.4
- net GND: now also C10.1, C9.1, CAN1.1, D12.1, D13.1, IC6.3, IC7.3, Q11.2, Q9.2, R34.2, R41.2, X1.2, X6.1; no longer U$7.10, U$8.10
- net PIN2: now also CAN1.2
- net PIN7: now also CAN1.3
- net PRECHARGE_EN_1: now also D13.3, R48.2, U$1.17/A3
- net PRECHARGE_EN_2: now also D12.3, R49.2, U$1.16/A2
Routing:
- net +5V: track 277.1 -> 412.2 mm, vias 9 -> 14
- net PRECHARGE_EN_2: track 2.75 -> 97.9 mm, vias 0 -> 2
- net PRECHARGE_EN_1: track 2.75 -> 94.7 mm, vias 0 -> 2
- net VCC: track 109.5 -> 33.3 mm
- net 5V: track 96.4 -> 36.4 mm
- net CHARGE_2: track 30.8 -> 78.4 mm, vias 0 -> 2
- net CONTACTOR_GND: track 0.00 -> 45.7 mm
- net CHARGE_1: track 33.9 -> 76.1 mm
- net PIN7: track 19.9 -> 49.6 mm
- net PIN2: track 24.0 -> 48.1 mm
- net CONTACT_EN_2: track 2.75 -> 22.3 mm
- net N$41: track 12.6 -> 30.3 mm
- net CONTACT_EN_1: track 2.75 -> 19.6 mm
- net N$36: track 0.00 -> 14.8 mm
- net N$47: track 0.00 -> 14.3 mm
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Other:
- board text added: "12V IN"
- board text added: "5V"
- board text added: "96V+"
- board text added: "APA102"
- board text added: "CONTACT EN"
- board text added: "EN"
- board text added: "EN1"
- board text added: "EN2"
- board text added: "PC1"
- board text added: "PC2"
- board text added: "PRE CHG EN"
- board text added: "PRECHARGE R1"
- board text added: "PRECHARGE R2"
- board text added: "PWR"
- board text added: "Pack Control Rev. 1"
- board text added: "RE+"
- board text added: "RE-"
- board text removed: "12V SUPPLY"
- board text removed: "FANS PWM"
- board text removed: "PRECHARGE R"
- board text removed: "Pack Controller Rev. 1"
- board text removed: "R+"
- board text removed: "R-"
