File: CANShield/CANShield.sch (EAGLE design)
At the start: 31 parts, among them Q1 16MHz, U2 ARDUINO_R3_SHIELD, U4 MCP2515, U5 MCP2551, X1 DB9 Plug

Commit message: Can shield
Parts:
- removed C7: 22pF, SparkFun-Capacitors:22PF-50V-5%(0603)
- removed CONTACTOR, CONTACTOR2, LEDS, PACKV: MSTBA2, con-phoenix-508:MSTBA2
- removed D3, D7: BAS40-04, diode:BAS40-04
- removed F2: PTCTHERMISTOR1206, SparkFun-PowerIC:PTCTHERMISTOR1206
- removed S2: RESET, SparkFun-Electromechanical:SWITCH-MOMENTARY-2SMD
- removed U2: ARDUINO_R3_SHIELD, SparkFun-Boards:ARDUINO_R3_SHIELD
- removed U4: MCP2515, SparkFun-DigitalIC:MCP2510SO
- added F3: 1812L, ptc-littlefuse:1812L
- added FANS, ON: MSTBA3, con-phoenix-508:MSTBA3
- added FAN_LEDS, GAUGES_APA102, PACK_LEDS: MSTBA4, con-phoenix-508:MSTBA4
- added IC1: 7805DT, linear:7805DT
- added IC2: 74LVC2G125DCT, 74xx-little-de:74LVC2G125DCT
- added J2: POWERPOLE_POWER25A_HORIZONTAL_G2, powerpoles:POWERPOLE_POWER25A_HORIZONTAL_G2
- added PRECHG1, PRECHG2: (no value), SparkFun-Connectors:M06POLAR
- added Q2, Q3, Q4, Q5, Q6: MOSFET-NCHANNELFDD8780, SparkFun-DiscreteSemi:MOSFET-NCHANNELFDD8780
- added Q7: MOSFET-NCHANNELBSS123LT1G, SparkFun-DiscreteSemi:MOSFET-NCHANNELBSS123LT1G
- added Q8: BSS123, transistor-small-signal:BSS123
- added R11, R15, R17, R19, R21, R23, R24, R25, R26, R27, R28, R8: 10K, SparkFun-Resistors:RESISTOR0603-RES
- added R14, R16, R18, R20, R6, R7, R9: 100R, SparkFun-Resistors:RESISTOR0603-RES
- added R22, R31, R32: (no value), SparkFun-Passives:RESISTOR0603-RES
- added R29: 100R, SparkFun-Passives:RESISTOR0603-RES
- added R30: 10K, SparkFun-Passives:RESISTOR0603-RES
- added R4: 100K, SparkFun-Resistors:RESISTOR0603-RES
- added SBO_1, SBO_2: (no value), adafruit:JST_2PIN-THM-RA
- added SG1: BUZZERNS, SparkFun-Electromechanical:BUZZERNS
- added U$1: TEENSY_3.0_BASIC-PGM, Teensy3.0:TEENSY_3.0_BASIC-PGM
- added U$2: F6136TR-ND, ptc-littlefuse:1812L
- C1: value 0.1uF -> (none); device SparkFun-Capacitors:0.1UF-25V(+80/-20%)(0603) -> SparkFun-Capacitors:CAP_POL1206
- C4: value 4.7uF -> (none); device SparkFun-Capacitors:4.7UF-6.3V-10%(0603)0603 -> SparkFun-Capacitors:CAP_POL1206
- C5: value 22pF -> (none); device SparkFun-Capacitors:22PF-50V-5%(0603) -> SparkFun-Capacitors:CAP0603-CAP
- D1: value MBRA140 -> (none); device SparkFun-DiscreteSemi:MBRA140 -> SparkFun-LED:LED1206
- D2: value BAS40-04 -> 250mA/100V; device diode:BAS40-04 -> SparkFun-DiscreteSemi:DIODEBAS16
- F1: value PTCTHERMISTOR1206 -> 1812L; device SparkFun-PowerIC:PTCTHERMISTOR1206 -> ptc-littlefuse:1812L
- Q1: value 16MHz -> MOSFET-NCHANNELFDD8780; device SparkFun-FreqCtrl:CRYSTAL5X3 -> SparkFun-DiscreteSemi:MOSFET-NCHANNELFDD8780
- R1, R5: value (none) -> 10K
- R2: value 100R -> 100K
Connections:
- removed net 12V: C4.1, D1.C, U2.VIN
- removed net 3.3V: U2.3.3V
- removed net A0: D7.C1A2, R2.1, U2.A0
- removed net AREF: U2.AREF
- removed net CAN_CS: U2.*D10, U4>NAME.CS
- removed net CAN_INT: U2.D2, U4>NAME.INT
- removed net CONTACT_SENSE_1: CONTACTOR2-1.1, D3.C1A2, R5.2, U2.*D9
- removed net CONTACT_SENSE_2: CONTACTOR-1.1, D2.C1A2, R1.2, U2.D8
- removed net D3: U2.*D3
- removed net D4: U2.D4
- removed net D5: U2.*D5
- removed net MISO: U2.D12, U4>NAME.SO
- removed net MOSI: U2.*D11, U4>NAME.SI
- removed net RS: S2.2, U2.RES, U4>NAME.RESET
- removed net RX: U2.RX
- removed net SCK: U2.D13, U4>NAME.SCK
- removed net TX: U2.TX
- new net +12V: F1.2, F3.2, FANS-1.1, J2.V+, ON-1.1, PRECHG1.2, PRECHG2.2, U$2.1
- new net +5V: C1.+, C5.1, C6.2, D2.C, IC1.VO, IC2G$3.VCC, R22.2, SG1.1, U$1.VIN, U5.VDD
- new net ACTIVE_1: PRECHG1.4, R24.1, U$1.17/A3
- new net ACTIVE_2: PRECHG2.4, R27.1, U$1.14/A0
- new net BUZZER: R29.1, U$1.20/A6
- new net CHARGED_1: PRECHG1.5, R25.1, U$1.18/A4
- new net CHARGED_2: PRECHG2.5, R28.1, U$1.15/A1
- new net CHARGING_1: PRECHG1.6, R23.1, U$1.19/A5
- new net CHARGING_2: PRECHG2.6, R26.1, U$1.16/A2
- new net FANS_B: R20.1, U$1.9
- new net FANS_G: R18.1, U$1.6
- new net FANS_R: R16.1, U$1.5
- new net FAN_PWM: R31.1, U$1.10
- new net LED_C: IC2G$2.I, U$1.13
- new net N$11: PACK_LEDS-4.1, Q3.D
- new net N$12: Q1.G, R7.2, R8.2
- new net N$15: Q3.G, R14.2, R15.2
- new net N$19: F3.1, FAN_LEDS-1.1
- new net N$20: FAN_LEDS-2.1, Q4.D
- new net N$21: FAN_LEDS-3.1, Q5.D
- new net N$22: FAN_LEDS-4.1, Q6.D
- new net N$23: Q4.G, R16.2, R17.2
- new net N$24: Q5.G, R18.2, R19.2
- new net N$25: Q6.G, R20.2, R21.2
- new net N$26: Q7.G, R29.2, R30.2
- new net N$27: Q8.G, R31.2, R32.2
- new net N$28: FANS-3.1, Q8.D
- new net N$29: GAUGES_APA102-1.1, U$2.2
- new net N$4: R4.2, SBO_2.2
- new net N$5: GAUGES_APA102-4.1, R6.1
- new net N$6: PACK_LEDS-2.1, Q1.D
- new net N$7: F1.1, PACK_LEDS-1.1
- new net N$8: PACK_LEDS-3.1, Q2.D
- new net PACK_B: R14.1, U$1.23/A9
- new net PACK_G: R9.1, U$1.22/A8
- new net PACK_R: R7.1, U$1.21/A7
- new net SBO_SENSE_1: R1.2, R4.1, U$1.7
- new net SBO_SENSE_2: R2.1, R5.2, U$1.8
- new net VCC: C4.+, IC1.VI, ON-2.1
- net 5V: now also PRECHG1.3, PRECHG2.3, R1.1, R23.2, R24.2, R25.2, R26.2, R27.2, R28.2, R5.1; no longer C1.2, C6.2, D2.C2, D3.C2, D7.C2, F2.2, U2.5V, U4P.VDD, U5.VDD
- net CAN_RXD: now also U$1.4; no longer U4>NAME.RXCAN
- net CAN_TXD: now also U$1.3; no longer U4>NAME.TXCAN
- net GND: now also C1.-, C4.-, C5.2, D1.C, FANS-2.1, GAUGES_APA102-2.1, IC1.GND, IC2G$1.OE, IC2G$2.OE, IC2G$3.GND, J2.GND, ON-3.1, PRECHG1.1, PRECHG2.1, Q1.S, Q2.S, Q3.S, Q4.S, Q5.S, Q6.S, Q7.S, Q8.S, R11.1, R15.1, R17.1, R19.1, R21.1, R30.1, R32.1, R8.1, U$1.AGND, U$1.GND; no longer C1.1, C4.2, C5.1, C7.1, D2.A1, D3.A1, D7.A1, LEDS-1.1, PACKV-2.1, R1.1, R5.1, S2.1, U2.GND@0, U2.GND@1, U2.GND@2, U4P.VSS
- net LED_D: now also IC2G$1.I, U$1.11; no longer R3.2, U2.SDA
- net N$1: now also SBO_1.2; no longer PACKV-1.1
- net N$13: now also Q2.G, R11.2, R9.2; no longer F1.2, X1.9
- net N$16: now also R22.1; no longer F1.1
- net N$17: now also IC2G$1.O, R3.2; no longer C7.2, Q1.2, U4>NAME.OSC1
- net N$18: now also D2.A, Q7.D, SG1.2; no longer C5.2, Q1.1, U4>NAME.OSC2
- net N$2: now also IC2G$2.O, R6.2; no longer CONTACTOR-2.1, CONTACTOR2-2.1, F2.1
- net N$3: now also GAUGES_APA102-3.1; no longer LEDS-2.1
Other:
- note added: "CAN Bus"
- note added: "Fan LED"
- note added: "Go to button/switch to turn system on"
- note added: "Pack LED"
- note removed: "Prosthesis Status Gauge"

Commit message: Most of the base board finished
Parts:
- removed PRECHG1, PRECHG2: (no value), SparkFun-Connectors:M06POLAR
- removed R23, R24, R25, R26, R27, R28: 10K, SparkFun-Resistors:RESISTOR0603-RES
- removed SBO_1, SBO_2: (no value), adafruit:JST_2PIN-THM-RA
- added D3, D4: BAS40-04, diode:BAS40-04
- added H1, H2, H3, H4: MOUNT-PAD-ROUND3.0, holes:MOUNT-PAD-ROUND3.0
- added IC3, IC4, IC5: ILD213T, SparkFun-DiscreteSemi:ILD213T
- added SBO_LOOP_1, SBO_LOOP_2: MSTBA2, con-phoenix-508:MSTBA2
- C1, C4: device SparkFun-Capacitors:CAP_POL1206 -> SparkFun-Capacitors:CAP_POLC
Connections:
- net +12V: no longer PRECHG1.2, PRECHG2.2
- net 5V: now also D3.C2, D4.C2; no longer PRECHG1.3, PRECHG2.3, R23.2, R24.2, R25.2, R26.2, R27.2, R28.2
- net ACTIVE_1: no longer PRECHG1.4, R24.1
- net ACTIVE_2: no longer PRECHG2.4, R27.1
- net BUZZER: now also U$1.23/A9; no longer U$1.20/A6
- net CHARGED_1: no longer PRECHG1.5, R25.1
- net CHARGED_2: no longer PRECHG2.5, R28.1
- net CHARGING_1: no longer PRECHG1.6, R23.1
- net CHARGING_2: no longer PRECHG2.6, R26.1
- net FANS_B: now also U$1.5; no longer U$1.9
- net FANS_R: now also U$1.9; no longer U$1.5
- net GND: now also D3.A1, D4.A1, H1.MOUNT, H2.MOUNT, H3.MOUNT, H4.MOUNT, SBO_LOOP_1-2.1, SBO_LOOP_2-2.1; no longer PRECHG1.1, PRECHG2.1
- net N$1: now also SBO_LOOP_2-1.1; no longer SBO_1.2
- net N$4: now also SBO_LOOP_1-1.1; no longer SBO_2.2
- net PACK_B: now also U$1.22/A8; no longer U$1.23/A9
- net PACK_G: now also U$1.21/A7; no longer U$1.22/A8
- net PACK_R: now also U$1.20/A6; no longer U$1.21/A7
- net SBO_SENSE_1: now also D3.C1A2
- net SBO_SENSE_2: now also D4.C1A2

Commit message: precharge progress
Parts:
- removed IC4, IC5: ILD213T, SparkFun-DiscreteSemi:ILD213T
- added 74HC125M: MM74HC125M, Fairchild_By_element14_Batch_1:MM74HC125M
- added D10, D11, D6, D7: (no value), SparkFun-DiscreteSemi:DIODESOD123
- added LM393M: LM393M, Fairchild_By_element14_Batch_1:LM393M
- added PRECHARGE_FUSE: FUSEX20MM, SparkFun-Passives:FUSEX20MM
- added PRECHARGE_RELAY, PRECHARGE_RELAY1: DS2Y-S-DC5V, relay:DS2Y-S-DC5V
- added Q11, Q13, Q14, Q9: IRLML6344TRPBF, SparkFun-DiscreteSemi:MOSFET-NCHANNELBSS123LT1G
- added R23, R24, R25, R26: 10K, SparkFun-Passives:RESISTOR0603-RES
- added R33, R45: 100k, SparkFun-Resistors:RESISTOR0603-RES
- added R34, R41, R46, R47: 10k, SparkFun-Resistors:RESISTOR0603-RES
- added R36, R37, R42: 470k, SparkFun-Resistors:RESISTOR0805-RES
- added R38, R43: 13K, SparkFun-Resistors:RESISTOR0805-RES
- added R39: 110k, SparkFun-Resistors:RESISTOR0805-RES
- added R40: 12K, SparkFun-Resistors:RESISTOR0805-RES
- added U$5: REE-0505S, grant:REE-0505S
- added U$7, U$8: RELAY-2G5Q, SparkFun-Electromechanical:RELAY-2G5Q
- added X2, X3, X4, X5: SMKDSP_1,5/2, con-phoenix-smkdsp:SMKDSP_1,5/2
- FANS, ON: value MSTBA3 -> SMKDSP_1,5/3; device con-phoenix-508:MSTBA3 -> con-phoenix-smkdsp:SMKDSP_1,5/3
- FAN_LEDS, GAUGES_APA102, PACK_LEDS: value MSTBA4 -> SMKDSP_1,5/4; device con-phoenix-508:MSTBA4 -> con-phoenix-smkdsp:SMKDSP_1,5/4
- SBO_LOOP_1, SBO_LOOP_2: value MSTBA2 -> SMKDSP_1,5/2; device con-phoenix-508:MSTBA2 -> con-phoenix-smkdsp:SMKDSP_1,5/2
Connections:
- removed net CHARGED_1: U$1.18/A4
- removed net CHARGING_1: U$1.19/A5
- new net 96V_IN_FUSED: PRECHARGE_FUSE.1, PRECHARGE_RELAY12.S, PRECHARGE_RELAY2.S, R37.2
- new net CAP_CHARGE_REF: LM393M.IN1_(-), R39.1, R40.2
- new net CAP_CHARGE_V_CURR_1: LM393M.IN1_(+), R36.1, R38.2
- new net CAP_CHARGE_V_CURR_2: R42.1, R43.2
- new net CHARGE_1: IC3.CT1, R23.1, U$1.19/A5
- new net CHARGE_2: IC3.CT2, R26.1, U$1.18/A4
- new net CHARGE_ISO_1: 74HC125M.Y1, R25.2
- new net CHARGE_ISO_2: 74HC125M.Y2, R24.2
- new net CONTACT_EN_1: Q13.G, R46.1
- new net CONTACT_EN_2: Q14.G, R47.1
- new net GNDI: IC3.C1, IC3.C2, U$5.-VOUT, X4-2.KL
- new net N$30: R37.1, R39.2
- new net N$31: 74HC125M.A3, 74HC125M.A4, LM393M.OUT2, R45.2
- new net N$32: IC3.A2, R25.1
- new net N$33: D10.A, Q14.D, U$8.9
- new net N$34: IC3.A1, R24.1
- new net N$35: D11.A, Q13.D, U$7.9
- new net N$36: 74HC125M.Y3
- new net N$37: 74HC125M.Y4
- new net N$38: U$7.5, U$7.6
- new net N$39: U$8.5, U$8.6
- new net N$40: PRECHARGE_RELAY3.P, X2-1.KL
- new net N$41: PRECHARGE_RELAY13.P, X3-1.KL
- new net N$42: PRECHARGE_FUSE.2, X4-1.KL
- new net PRECHARGE_EN_1: Q9.G, R34.1
- new net PRECHARGE_EN_2: Q11.G, R41.1
- new net PRECHARGE_OUT_1: PRECHARGE_RELAY2.O, PRECHARGE_RELAY3.S, R36.2, X5-1.KL
- new net PRECHARGE_OUT_2: PRECHARGE_RELAY12.O, PRECHARGE_RELAY13.S, R42.2, X5-2.KL
- new net PRECHARGE_RESISTOR_IN: PRECHARGE_RELAY2.P, X2-2.KL
- new net PRECHARGE_RESISTOR_IN1: PRECHARGE_RELAY12.P, X3-2.KL
- new net PRECH_DRAIN: D6.A, PRECHARGE_RELAY1.-, Q9.D
- new net PRECH_DRAIN1: D7.A, PRECHARGE_RELAY11.-, Q11.D
- new net PRECH_STATE_TO_BUFF: 74HC125M.A1, 74HC125M.A2, LM393M.OUT1, R33.2
- net +12V: now also D10.C, D11.C, FANS-1.KL, ON-1.KL, U$7.2, U$8.2; no longer FANS-1.1, ON-1.1
- net +5V: now also R23.2, R26.2, U$5.+VIN
- net 5V: now also 74HC125M.VCC, D6.C, D7.C, LM393M.VCC, PRECHARGE_RELAY1.+, PRECHARGE_RELAY11.+, R33.1, R45.1, U$5.+VOUT
- net BUZZER: now also U$1.10; no longer U$1.23/A9
- net FAN_PWM: now also U$1.23/A9; no longer U$1.10
- net GND: now also 74HC125M.C1, 74HC125M.C2, 74HC125M.C3, 74HC125M.C4, 74HC125M.GND, FANS-2.KL, GAUGES_APA102-2.KL, IC3.ET1, IC3.ET2, LM393M.GND, ON-3.KL, PRECHARGE_RELAY13.O, PRECHARGE_RELAY3.O, Q11.S, Q13.S, Q14.S, Q9.S, R34.2, R38.1, R40.1, R41.2, R43.1, R46.2, R47.2, SBO_LOOP_1-2.KL, SBO_LOOP_2-2.KL, U$5.-VIN, U$7.10, U$8.10; no longer FANS-2.1, GAUGES_APA102-2.1, ON-3.1, SBO_LOOP_1-2.1, SBO_LOOP_2-2.1
- net N$1: now also SBO_LOOP_2-1.KL; no longer SBO_LOOP_2-1.1
- net N$11: now also PACK_LEDS-4.KL; no longer PACK_LEDS-4.1
- net N$19: now also FAN_LEDS-1.KL; no longer FAN_LEDS-1.1
- net N$20: now also FAN_LEDS-2.KL; no longer FAN_LEDS-2.1
- net N$21: now also FAN_LEDS-3.KL; no longer FAN_LEDS-3.1
- net N$22: now also FAN_LEDS-4.KL; no longer FAN_LEDS-4.1
- net N$28: now also FANS-3.KL; no longer FANS-3.1
- net N$29: now also GAUGES_APA102-1.KL; no longer GAUGES_APA102-1.1
- net N$3: now also GAUGES_APA102-3.KL; no longer GAUGES_APA102-3.1
- net N$4: now also SBO_LOOP_1-1.KL; no longer SBO_LOOP_1-1.1
- net N$5: now also GAUGES_APA102-4.KL; no longer GAUGES_APA102-4.1
- net N$6: now also PACK_LEDS-2.KL; no longer PACK_LEDS-2.1
- net N$7: now also PACK_LEDS-1.KL; no longer PACK_LEDS-1.1
- net N$8: now also PACK_LEDS-3.KL; no longer PACK_LEDS-3.1
- net VCC: now also ON-2.KL; no longer ON-2.1
Other:
- note added: "*Output goes HIGH (5V) when cap charge goes ABOVE reference"
- note added: "Part #1A3399-10 from Mouser. Must order in multiples of 2"

Commit message: down to one airwire
Parts:
- removed X1: DB9 Plug, SparkFun-Connectors:DB9MALE
- added CAN: SMKDSP_1,5/3, con-phoenix-smkdsp:SMKDSP_1,5/3
- added CONTACTOR_1, CONTACTOR_2: SMKDSP_1,5/4, con-phoenix-smkdsp:SMKDSP_1,5/4
- added D8, D9: BAS40-04, diode:BAS40-04
- added PF1, PF2: PTC-2920L, polyswitch:PTC-2920L
- added R27, R28: 10K, SparkFun-Resistors:RESISTOR0603-RES
- added R35, R44: 100K, SparkFun-Resistors:RESISTOR0603-RES
- F1, F3: value 1812L -> PTC-2920L; device ptc-littlefuse:1812L -> polyswitch:PTC-2920L
- U$2: device ptc-littlefuse:1812L -> polyswitch:PTC-2920L
Connections:
- removed net ACTIVE_1: U$1.17/A3
- removed net ACTIVE_2: U$1.14/A0
- removed net CHARGED_2: U$1.15/A1
- removed net CHARGING_2: U$1.16/A2
- removed net GNDI: IC3.C1, IC3.C2, U$5.-VOUT, X4-2.KL
- removed net N$36: 74HC125M.Y3
- removed net N$37: 74HC125M.Y4
- removed net NC1: X1.1
- removed net NC2: X1.4
- removed net NC3: X1.6
- removed net NC5: X1.8
- new net AGND: 74HC125M.C1, 74HC125M.C2, 74HC125M.C3, 74HC125M.C4, 74HC125M.GND, IC3.C1, IC3.C2, LM393M.GND, PRECHARGE_RELAY13.O, PRECHARGE_RELAY3.O, Q11.S, Q9.S, R34.2, R38.1, R40.1, R41.2, R43.1, U$5.-VOUT, X4-2.KL
- new net CONTACTOR_CLOSED_SENSE_1: D8.C1A2, R27.2, R44.1, U$1.16/A2
- new net CONTACTOR_CLOSED_SENSE_2: D9.C1A2, R28.2, R35.1, U$1.17/A3
- new net N$43: CONTACTOR_1-4.KL, PF2.2
- new net N$44: CONTACTOR_2-4.KL, PF1.2
- new net N$45: CONTACTOR_2-2.KL, R35.2
- new net N$46: CONTACTOR_1-2.KL, R44.2
- net +12V: now also PF1.1, PF2.1
- net +5V: now also D3.C2, D4.C2, D8.C2, D9.C2, R1.1, R27.1, R28.1, R5.1
- net 5V: no longer D3.C2, D4.C2, R1.1, R5.1
- net CAP_CHARGE_REF: now also LM393M.IN2_(-)
- net CAP_CHARGE_V_CURR_2: now also LM393M.IN2_(+)
- net CHARGE_1: now also U$1.15/A1; no longer U$1.19/A5
- net CHARGE_2: now also U$1.14/A0; no longer U$1.18/A4
- net CHARGE_ISO_2: now also 74HC125M.Y3; no longer 74HC125M.Y2
- net GND: now also CAN-1.KL, CONTACTOR_1-1.KL, CONTACTOR_2-1.KL, D8.A1, D9.A1; no longer 74HC125M.C1, 74HC125M.C2, 74HC125M.C3, 74HC125M.C4, 74HC125M.GND, LM393M.GND, PRECHARGE_RELAY13.O, PRECHARGE_RELAY3.O, Q11.S, Q9.S, R34.2, R38.1, R40.1, R41.2, R43.1, X1.3
- net N$38: now also CONTACTOR_1-3.KL
- net N$39: now also CONTACTOR_2-3.KL
- net PIN2: now also CAN-2.KL; no longer X1.2
- net PIN7: now also CAN-3.KL; no longer X1.7

Commit message: Mostly done
Parts:
- C1, C4: value (none) -> 10uF
- C5: value (none) -> 0.1uF
- R22: value (none) -> 470R
- R31: value (none) -> 100R
- R32: value (none) -> 10K
Connections:
- net PRECHARGE_RESISTOR_IN renamed PRECHARGE_RESISTOR_IN_1
- net PRECHARGE_RESISTOR_IN1 renamed PRECHARGE_RESISTOR_IN_2
Other:
- moved on the sheet: X3-1
Changed lines of the file:
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@@
 <part name="GND2" library="SparkFun-Aesthetics" deviceset="GND" device=""/>
 <part name="IC1" library="linear" deviceset="78*" device="DT" technology="05"/>
-<part name="C1" library="SparkFun-Capacitors" deviceset="CAP_POL" device="C"/>
-<part name="C4" library="SparkFun-Capacitors" deviceset="CAP_POL" device="C"/>
+<part name="C1" library="SparkFun-Capacitors" deviceset="CAP_POL" device="C" value="10uF"/>
+<part name="C4" library="SparkFun-Capacitors" deviceset="CAP_POL" device="C" value="10uF"/>
 <part name="GND1" library="SparkFun-Aesthetics" deviceset="GND" device=""/>
 <part name="GND6" library="SparkFun-Aesthetics" deviceset="GND" device=""/>
@@
 <part name="D1" library="SparkFun-LED" deviceset="LED" device="1206"/>
 <part name="GND29" library="SparkFun-Aesthetics" deviceset="GND" device=""/>
-<part name="R22" library="SparkFun-Passives" deviceset="RESISTOR" device="0603-RES"/>
+<part name="R22" library="SparkFun-Passives" deviceset="RESISTOR" device="0603-RES" value="470R"/>
 <part name="ON" library="con-phoenix-smkdsp" deviceset="SMKDSP_1,5/3" device=""/>
 <part name="GND3" library="SparkFun-Aesthetics" deviceset="GND" device=""/>
@@
 <part name="GND19" library="SparkFun-Aesthetics" deviceset="GND" device=""/>
 <part name="GND32" library="SparkFun-Aesthetics" deviceset="GND" device=""/>
-<part name="C5" library="SparkFun-Capacitors" deviceset="CAP" device="0603-CAP"/>
+<part name="C5" library="SparkFun-Capacitors" deviceset="CAP" device="0603-CAP" value="0.1uF"/>
 <part name="GND33" library="SparkFun-Aesthetics" deviceset="GND" device=""/>
 <part name="SG1" library="SparkFun-Electromechanical" deviceset="BUZZER" device="NS"/>
@@
 <part name="GND35" library="supply1" deviceset="GND" device=""/>
 <part name="Q8" library="transistor-small-signal" deviceset="BSS123" device=""/>
-<part name="R31" library="SparkFun-Passives" deviceset="RESISTOR" device="0603-RES"/>
-<part name="R32" library="SparkFun-Passives" deviceset="RESISTOR" device="0603-RES"/>
+<part name="R31" library="SparkFun-Passives" deviceset="RESISTOR" device="0603-RES" value="100R"/>
+<part name="R32" library="SparkFun-Passives" deviceset="RESISTOR" device="0603-RES" value="10K"/>
 <part name="GND36" library="supply1" deviceset="GND" device=""/>
 <part name="GND37" library="supply1" deviceset="GND" device=""/>
@@
 <instance part="R6" gate="G$1" x="30.48" y="137.16" rot="R180"/>
 <instance part="GND2" gate="1" x="-55.88" y="198.12" rot="R90"/>
-<instance part="P+1" gate="1" x="-58.42" y="205.74"/>
+<instance part="P+1" gate="1" x="-48.26" y="205.74"/>
 <instance part="U$1" gate="G$1" x="-81.28" y="187.96"/>
 <instance part="GND7" gate="1" x="-60.96" y="195.58" rot="R90"/>
@@
 <net name="+5V" class="0">
 <segment>
-<wire x1="-66.04" y1="203.2" x2="-58.42" y2="203.2" width="0.1524" layer="91"/>
+<wire x1="-66.04" y1="203.2" x2="-48.26" y2="203.2" width="0.1524" layer="91"/>
 <pinref part="P+1" gate="1" pin="+5V"/>
 <pinref part="U$1" gate="G$1" pin="VIN"/>
@@
 <instance part="X2" gate="-1" x="0" y="157.48"/>
 <instance part="X2" gate="-2" x="0" y="177.8"/>
-<instance part="X3" gate="-1" x="-2.54" y="50.8"/>
+<instance part="X3" gate="-1" x="10.16" y="30.48"/>
 <instance part="X3" gate="-2" x="-2.54" y="71.12"/>
 <instance part="X4" gate="-1" x="-109.22" y="195.58"/>
@@
 </segment>
 </net>
-<net name="PRECHARGE_RESISTOR_IN" class="0">
+<net name="PRECHARGE_RESISTOR_IN_1" class="0">
 <segment>
 <pinref part="PRECHARGE_RELAY" gate="2" pin="P"/>
@@
 </segment>
 </net>
-<net name="PRECHARGE_RESISTOR_IN1" class="0">
+<net name="PRECHARGE_RESISTOR_IN_2" class="0">
 <segment>
 <pinref part="PRECHARGE_RELAY1" gate="2" pin="P"/>
@@
 <pinref part="PRECHARGE_RELAY1" gate="3" pin="P"/>
 <pinref part="X3" gate="-1" pin="KL"/>
-<wire x1="2.54" y1="50.8" x2="15.24" y2="50.8" width="0.1524" layer="91"/>
-</segment>
-</net>
+<wire x1="15.24" y1="30.48" x2="15.24" y2="50.8" width="0.1524" layer="91"/>
+</segment>
+</net>

Commit message: Feature complete pcb
Parts:
- added C10, C9: 0.1uF, SparkFun-Capacitors:CAP0603-CAP
- added CAN1: SMKDSP_1,5/3, con-phoenix-smkdsp:SMKDSP_1,5/3
- added D12, D13: BAS40-04, diode:BAS40-04
- added F2: PTCTHERMISTOR1206, SparkFun-PowerIC:PTCTHERMISTOR1206
- added IC6, IC7: 74LVC1G04DBV, 74xx-little-de:74LVC1G04DBV
- added R48, R49: 100R, SparkFun-Passives:RESISTOR0603-RES
- added X1: SMKDSP_1,5/2, con-phoenix-smkdsp:SMKDSP_1,5/2
- added X6: SMKDSP_1,5/4, con-phoenix-smkdsp:SMKDSP_1,5/4
Connections:
- new net CONTACTOR_GND: U$7.10, U$8.10, X1-1.KL
- new net N$36: R48.1, X6-4.KL
- new net N$37: R49.1, X6-3.KL
- new net N$47: F2.1, X6-2.KL
- net +5V: now also C10.2, C9.2, D12.C2, D13.C2, D6.C, D7.C, F2.2, IC6P.VCC, IC7P.VCC, PRECHARGE_RELAY1.+, PRECHARGE_RELAY11.+
- net 5V: no longer D6.C, D7.C, PRECHARGE_RELAY1.+, PRECHARGE_RELAY11.+
- net AGND: no longer Q11.S, Q9.S, R34.2, R41.2
- net CHARGE_1: now also IC6A.I, U$1.14/A0; no longer U$1.15/A1
- net CHARGE_2: now also IC7A.I, U$1.15/A1; no longer U$1.14/A0
- net CONTACTOR_CLOSED_SENSE_1: now also U$1.18/A4; no longer U$1.16/A2
- net CONTACTOR_CLOSED_SENSE_2: now also U$1.19/A5; no longer U$1.17/A3
- net CONTACT_EN_1: now also IC6A.O
- net CONTACT_EN_2: now also IC7A.O
- net GND: now also C10.1, C9.1, CAN1-1.KL, D12.A1, D13.A1, IC6P.GND, IC7P.GND, Q11.S, Q9.S, R34.2, R41.2, X1-2.KL, X6-1.KL; no longer U$7.10, U$8.10
- net PIN2: now also CAN1-2.KL
- net PIN7: now also CAN1-3.KL
- net PRECHARGE_EN_1: now also D13.C1A2, R48.2, U$1.17/A3
- net PRECHARGE_EN_2: now also D12.C1A2, R49.2, U$1.16/A2
Other:
- moved on the sheet: D6, D7, PRECHARGE_RELAY, PRECHARGE_RELAY1, Q11, Q9, R34, R36, R38, R41, R42, R43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
