File: can-pump/CANShield.sch (EAGLE design)
At the start: 109 parts, among them IC2 MC1525TT, IC3 QUAD_OPAMPD, J1 POWERPOLE_POWER25A_HORIZONTAL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, K1 G5LE, K2 G5LE, K3 G5LE, K4 G5LE, K5 G5LE, K6 G5LE, K7 G5LE, K8 G5LE, Q1 MOSFET-NCHANNELAO3404A, Q2 MOSFET-NCHANNELAO3404A, Q3 MOSFET-NCHANNELAO3404A, Q4 MOSFET-NCHANNELAO3404A, Q5 MOSFET-NCHANNELAO3404A, Q6 MOSFET-NCHANNELAO3404A, Q7 MOSFET-NCHANNELAO3404A, Q8 MOSFET-NCHANNELAO3404A, U5 MCP2551, X2 SMKDSP_1,5/2, X5 SMKDSP_1,5/2, X6 SMKDSP_1,5/2, X7 SMKDSP_1,5/2, X8 SMKDSP_1,5/2

Commit message: Latest
Parts:
- removed D10, D12, D14, D16, D18, D3, D6, D8: (no value), SparkFun-LED:LED1206
- removed R15, R18, R21, R25, R28, R3, R6, R9: 1K, SparkFun-Passives:RESISTOR0603-RES
- added D24, D26: (no value), adafruit:DIODESOD-123
- added K10, K9: G5LE, relay:G5LE
- added Q10, Q9: MOSFET-NCHANNELAO3404A, SparkFun-DiscreteSemi:MOSFET-NCHANNELAO3404A
- added R45, R48: 100R, SparkFun-Passives:RESISTOR0603-RES
- added R46, R49: 10K, SparkFun-Passives:RESISTOR0603-RES
- added U$10, U$11, U$12, U$2, U$4, U$5, U$6, U$7, U$8, U$9: FUSE, grant:FUSE
- added X1, X3, X4, X9: SMKDSP_1,5/3, con-phoenix-smkdsp:SMKDSP_1,5/3
- added X10, X11, X12, X13, X14, X15: SMKDSP_1,5/2, con-phoenix-smkdsp:SMKDSP_1,5/2
Connections:
- removed net 5V: D20.C2, D21.C2, D22.C2, D23.C2
- removed net N$11: D6.A, R6.1
- removed net N$17: D8.A, R9.1
- removed net N$21: D10.A, R15.1
- removed net N$25: D12.A, R18.1
- removed net N$29: D14.A, R21.1
- removed net N$33: D16.A, R25.1
- removed net N$37: D18.A, R28.1
- removed net N$5: D3.A, R3.1
- new net N$15: K62.S, U$9.A
- new net N$20: R44.1, X9-1.KL
- new net N$24: R42.1, X3-1.KL
- new net N$28: R43.1, X4-1.KL
- new net N$3: K32.S, U$7.A
- new net N$32: R41.1, X1-1.KL
- new net N$4: K42.S, U$8.A
- new net N$41: K22.S, U$4.A
- new net N$45: K82.S, U$5.A
- new net N$50: K72.S, U$2.A
- new net N$53: K12.S, U$6.A
- new net N$55: D24.A, K91.2, Q9.D
- new net N$57: Q9.G, R45.2, R46.2
- new net N$59: D26.A, K101.2, Q10.D
- new net N$60: Q10.G, R48.2, R49.2
- new net N$62: K92.S, U$11.A
- new net N$63: K102.S, U$12.A
- new net N$65: U$5.B, X13-1.KL
- new net N$66: U$4.B, X11-1.KL
- new net N$67: U$6.B, X10-1.KL
- new net N$68: U$9.B, X6-1.KL
- new net N$69: K52.S, U$10.A
- new net N$70: U$7.B, X7-1.KL
- new net N$71: U$10.B, X5-1.KL
- new net N$72: U$12.B, X15-1.KL
- new net N$73: U$11.B, X14-1.KL
- new net N$8: U$8.B, X8-1.KL
- new net RELAY10: R48.1, U$1.22/A8
- new net RELAY9: R45.1, U$1.23/A9
- net +5V: now also D20.C2, D21.C2, D22.C2, D23.C2, X1-2.KL, X3-2.KL, X4-2.KL, X9-2.KL
- net GND: now also Q10.S, Q9.S, R46.1, R49.1, X1-3.KL, X10-2.KL, X11-2.KL, X12-2.KL, X13-2.KL, X14-2.KL, X15-2.KL, X3-3.KL, X4-3.KL, X5-2.KL, X6-2.KL, X7-2.KL, X8-2.KL, X9-3.KL
- net N$12: no longer D8.C
- net N$18: no longer D10.C
- net N$2: no longer D3.C
- net N$22: no longer D12.C
- net N$26: no longer D14.C
- net N$30: no longer D16.C
- net N$34: no longer D18.C
- net N$48: now also IC3D.+IN; no longer IC3A.+IN
- net N$51: now also IC3A.+IN; no longer IC3D.+IN
- net N$6: no longer D6.C
- net N$64: now also U$2.B, X12-1.KL; no longer D13.C, K61.1
- net VCC: now also D13.C, D24.C, D26.C, K101.1, K102.P, K61.1, K91.1, K92.P; no longer R15.2, R18.2, R21.2, R25.2, R28.2, R3.2, R6.2, R9.2
Other:
- moved on the sheet: D20, D23, R41, R44, X5-1, X5-2, X6-1, X6-2, X7-1, X7-2, X8-1, X8-2
